Commit message: Remove special urdf files for simulation and update configuration of unified files.

File: urdf/ur_macro.xacro (robot description, xacro)
@@ -59,4 +59,6 @@
     use_fake_hardware:=false
     fake_sensor_commands:=false
+    sim_gazebo:=false
+    sim_ignition:=false
     headless_mode:=false
     initial_positions:=${dict(shoulder_pan_joint=0.0,shoulder_lift_joint=-1.57,elbow_joint=0.0,wrist_1_joint=-1.57,wrist_2_joint=0.0,wrist_3_joint=0.0)}
@@ -81,4 +83,6 @@
       initial_positions="${initial_positions}"
       fake_sensor_commands="$(arg fake_sensor_commands)"
+      sim_gazebo="$(arg sim_gazebo)"
+      sim_ignition="$(arg sim_ignition)"
       headless_mode="$(arg headless_mode)"
       script_filename="$(arg script_filename)"
@@ -302,4 +306,10 @@
       <dynamics damping="0" friction="0"/>
     </joint>
+    <link name="${prefix}ft_frame"/>
+    <joint name="${prefix}wrist_3_link-ft_frame" type="fixed">
+      <parent link="${prefix}wrist_3_link"/>
+      <child link="${prefix}ft_frame"/>
+      <origin xyz="0 0 0" rpy="${pi} 0 0"/>
+    </joint>
     <!-- ROS-Industrial 'base' frame - base_link to UR 'Base' Coordinates transform -->
     <link name="${prefix}base"/>
